File: rf_controller_hw/rf_controller_hw.kicad_sch (KiCad schematic)
At the start: 13 parts, among them J1 NRF24L01, SW1 SW_Push, SW10 SW_SPDT, SW2 SW_Push, SW3 SW_Push, SW4 SW_Push, SW5 SW_DIP_x05, SW6 SW_Push, SW7 JOYSTICK_BUTTON, SW8 SW_Push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

Commit message: Fixed a bug in the first board:
Fixed bug in RP2040-Zero pinout
Added better logo
Re-added mounting holes
Switched to smaller joystick
Parts:
- RZ1: footprint rp2040-zero:RP2040-Zero -> rf_controller_hw:RP2040-Zero; symbol rp2040-zero:RP2040-Zero -> rf_controller_hw:RP2040-Zero
- SW5: renamed from SW7; footprint rf_controller_hw:Joystick_Button -> rf_controller_hw:ALPS_RKJXV1224
- renumbered SW5 to SW10, SW8 to SW7, SW9 to SW8, SW10 to SW9
Connections:
- net GND: now also RZ1.22 (GND); no longer RZ1.23 (GND)
- net SW1: now also RZ1.12 (GP11), SW1.2; no longer RZ1.6 (GP5), SW2.2
- net SW2: now also RZ1.10 (GP9), SW2.2; no longer RZ1.7 (GP6), SW1.2
- net SW3: now also RZ1.11 (GP10), SW3.2; no longer RZ1.8 (GP7), SW4.2
- net SW4: now also SW4.2; no longer SW3.2
- net SW6: now also RZ1.8 (GP7), SW6.2; no longer RZ1.11 (GP10), SW7.2
- net SW7: now also RZ1.7 (GP6), SW7.2; no longer RZ1.12 (GP11), SW8.2
- removed net SW5: RZ1.10 (GP9), SW6.2
- new net SW8: RZ1.6 (GP5), SW8.2
Changed lines of the file:
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@@
     (stroke (width 0) (type default) (color 0 0 0 0))
   )
-  (wire (pts (xy 111.76 109.22) (xy 117.602 109.22))
+  (wire (pts (xy 111.76 109.22) (xy 118.11 109.22))
     (stroke (width 0) (type default) (color 0 0 0 0))
   )
@@
     (stroke (width 0) (type default) (color 0 0 0 0))
   )
-  (wire (pts (xy 111.76 106.68) (xy 117.602 106.68))
+  (wire (pts (xy 111.76 106.68) (xy 118.11 106.68))
     (stroke (width 0) (type default) (color 0 0 0 0))
   )
@@
     (effects (font (size 1.27 1.27)) (justify left bottom))
   )
-  (label "SW6" (at 117.602 109.22 180)
-    (effects (font (size 1.27 1.27)) (justify right bottom))
+  (label "SW7" (at 69.85 101.6 0)
+    (effects (font (size 1.27 1.27)) (justify left bottom))
   )
   (label "SPI_SCK" (at 71.882 91.44 0)
@@
     (effects (font (size 1.27 1.27)) (justify left bottom))
   )
-  (label "SW7" (at 117.602 106.68 180)
-    (effects (font (size 1.27 1.27)) (justify right bottom))
+  (label "SW8" (at 69.85 99.06 0)
+    (effects (font (size 1.27 1.27)) (justify left bottom))
   )
   (label "JOY_Y" (at 119.38 88.9 180)
@@
     (effects (font (size 1.27 1.27)) (justify left bottom))
   )
-  (label "SW3" (at 74.93 153.67 0)
-    (effects (font (size 1.27 1.27)) (justify left bottom))
-  )
-  (label "SW5" (at 69.85 109.22 0)
+  (label "SW4" (at 74.93 153.67 0)
+    (effects (font (size 1.27 1.27)) (justify left bottom))
+  )
+  (label "SW6" (at 69.85 104.14 0)
     (effects (font (size 1.27 1.27)) (justify left bottom))
   )
@@
     (effects (font (size 1.27 1.27)) (justify left bottom))
   )
-  (label "SW7" (at 185.42 124.46 0)
-    (effects (font (size 1.27 1.27)) (justify left bottom))
-  )
-  (label "SW6" (at 171.45 124.46 0)
-    (effects (font (size 1.27 1.27)) (justify left bottom))
-  )
-  (label "SW4" (at 74.93 166.37 0)
-    (effects (font (size 1.27 1.27)) (justify left bottom))
-  )
-  (label "SW1" (at 74.93 137.16 0)
-    (effects (font (size 1.27 1.27)) (justify left bottom))
-  )
-  (label "SW4" (at 69.85 106.68 0)
-    (effects (font (size 1.27 1.27)) (justify left bottom))
+  (label "SW8" (at 185.42 124.46 0)
+    (effects (font (size 1.27 1.27)) (justify left bottom))
+  )
+  (label "SW7" (at 171.45 124.46 0)
+    (effects (font (size 1.27 1.27)) (justify left bottom))
+  )
+  (label "SW3" (at 74.93 166.37 0)
+    (effects (font (size 1.27 1.27)) (justify left bottom))
+  )
+  (label "SW2" (at 74.93 137.16 0)
+    (effects (font (size 1.27 1.27)) (justify left bottom))
+  )
+  (label "SW3" (at 118.11 109.22 180)
+    (effects (font (size 1.27 1.27)) (justify right bottom))
   )
   (label "SPI_MOSI" (at 69.342 93.98 0)
@@
     (effects (font (size 1.27 1.27)) (justify left bottom))
   )
-  (label "SW2" (at 74.93 151.13 0)
-    (effects (font (size 1.27 1.27)) (justify left bottom))
-  )
-  (label "SW5" (at 157.48 124.46 0)
-    (effects (font (size 1.27 1.27)) (justify left bottom))
-  )
-  (label "SW1" (at 69.85 99.06 0)
+  (label "SW1" (at 74.93 151.13 0)
+    (effects (font (size 1.27 1.27)) (justify left bottom))
+  )
+  (label "SW6" (at 157.48 124.46 0)
+    (effects (font (size 1.27 1.27)) (justify left bottom))
+  )
+  (label "SW2" (at 69.85 109.22 0)
     (effects (font (size 1.27 1.27)) (justify left bottom))
   )
@@
     (effects (font (size 1.27 1.27)) (justify left bottom))
   )
-  (label "SW3" (at 69.85 104.14 0)
+  (label "SW4" (at 69.85 106.68 0)
     (effects (font (size 1.27 1.27)) (justify left bottom))
   )
@@
     (effects (font (size 1.27 1.27)) (justify left bottom))
   )
-  (label "SW2" (at 69.85 101.6 0)
-    (effects (font (size 1.27 1.27)) (justify left bottom))
+  (label "SW1" (at 118.11 106.68 180)
+    (effects (font (size 1.27 1.27)) (justify right bottom))
   )
   (label "JOY_X" (at 119.38 86.36 180)
@@
     (pin "1")
   )
-  (symbol (lib_id "rp2040-zero:RP2040-Zero") (at 96.52 96.52 0) (unit 1)
-    (in_bom yes) (on_board yes) (fields_autoplaced)
-    (property "Reference" "RZ1" (id 0) (at 98.5394 113.665 0)
+  (symbol (lib_id "rf_controller_hw:RP2040-Zero") (at 96.52 96.52 0) (unit 1)
+    (in_bom yes) (on_board yes) (fields_autoplaced)
+    (property "Reference" "RZ1" (id 0) (at 98.5394 114.3 0)
       (effects (font (size 1.27 1.27)) (justify left))
     )
-    (property "Value" "RP2040-Zero" (id 1) (at 98.5394 116.205 0)
+    (property "Value" "RP2040-Zero" (id 1) (at 98.5394 116.84 0)
       (effects (font (size 1.27 1.27)) (justify left))
     )
-    (property "Footprint" "rp2040-zero:RP2040-Zero" (id 2) (at 98.5394 118.745 0)
+    (property "Footprint" "rf_controller_hw:RP2040-Zero" (id 2) (at 98.5394 119.38 0)
       (effects (font (size 1.27 1.27)) (justify left))
     )
@@
   (symbol (lib_id "Switch:SW_SPDT") (at 223.52 76.2 0) (unit 1)
     (in_bom yes) (on_board yes) (fields_autoplaced)
-    (property "Reference" "SW10" (id 0) (at 223.52 68.58 0))
+    (property "Reference" "SW9" (id 0) (at 223.52 68.58 0))
     (property "Value" "SW_SPDT" (id 1) (at 223.52 71.12 0))
     (property "Footprint" "Connector_PinHeader_2.54mm:PinHeader_1x03_P2.54mm_Vertical" (id 2) (at 223.52 76.2 0)
@@
   (symbol (lib_id "rf_controller_hw:JOYSTICK_BUTTON") (at 167.64 41.91 0) (unit 1)
     (in_bom yes) (on_board yes) (fields_autoplaced)
-    (property "Reference" "SW7" (id 0) (at 181.864 38.735 0)
+    (property "Reference" "SW5" (id 0) (at 181.61 38.735 0)
       (effects (font (size 1.524 1.524)) (justify left))
     )
-    (property "Value" "JOYSTICK_BUTTON" (id 1) (at 181.864 42.545 0)
+    (property "Value" "JOYSTICK_BUTTON" (id 1) (at 181.61 42.545 0)
       (effects (font (size 1.524 1.524)) (justify left))
     )
-    (property "Footprint" "rf_controller_hw:Joystick_Button" (id 2) (at 181.864 46.355 0)
+    (property "Footprint" "rf_controller_hw:ALPS_RKJXV1224" (id 2) (at 181.61 46.355 0)
       (effects (font (size 1.524 1.524)) (justify left))
     )
@@
   (symbol (lib_id "Switch:SW_DIP_x05") (at 133.35 99.06 0) (mirror x) (unit 1)
     (in_bom yes) (on_board yes) (fields_autoplaced)
-    (property "Reference" "SW5" (id 0) (at 133.35 86.36 0))
+    (property "Reference" "SW10" (id 0) (at 133.35 86.36 0))
     (property "Value" "SW_DIP_x05" (id 1) (at 133.35 88.9 0))
     (property "Footprint" "Button_Switch_THT:SW_DIP_SPSTx05_Slide_9.78x14.88mm_W7.62mm_P2.54mm" (id 2) (at 133.35 99.06 0)
@@
   (symbol (lib_id "Switch:SW_Push") (at 185.42 134.62 90) (unit 1)
     (in_bom yes) (on_board yes)
-    (property "Reference" "SW9" (id 0) (at 186.69 133.3499 90)
+    (property "Reference" "SW8" (id 0) (at 186.69 133.3499 90)
       (effects (font (size 1.27 1.27)) (justify right))
     )
@@
   (symbol (lib_id "Switch:SW_Push") (at 171.45 134.62 90) (unit 1)
     (in_bom yes) (on_board yes)
-    (property "Reference" "SW8" (id 0) (at 172.72 133.3499 90)
+    (property "Reference" "SW7" (id 0) (at 172.72 133.3499 90)
       (effects (font (size 1.27 1.27)) (justify right))
     )
@@
     )
     (path "/3f0ff5f5-bbb3-4ace-9d30-ca3c070010e5"
-      (reference "RZ1") (unit 1) (value "RP2040-Zero") (footprint "rp2040-zero:RP2040-Zero")
+      (reference "RZ1") (unit 1) (value "RP2040-Zero") (footprint "rf_controller_hw:RP2040-Zero")
     )
     (path "/811832fb-9434-4b8b-8daf-4885d7552e58"
@@
       (reference "SW4") (unit 1) (value "SW_Push") (footprint "Button_Switch_THT:SW_PUSH_6mm_H5mm")
     )
-    (path "/691fef37-3035-4bf1-a7e9-ebb9530ca238"
-      (reference "SW5") (unit 1) (value "SW_DIP_x05") (footprint "Button_Switch_THT:SW_DIP_SPSTx05_Slide_9.78x14.88mm_W7.62mm_P2.54mm")
+    (path "/4cdcdbcd-0741-4981-b73d-143743805270"
+      (reference "SW5") (unit 1) (value "JOYSTICK_BUTTON") (footprint "rf_controller_hw:ALPS_RKJXV1224")
     )
     (path "/0f228d33-5293-46e5-aa6b-af327a95a055"
       (reference "SW6") (unit 1) (value "SW_Push") (footprint "Button_Switch_THT:SW_PUSH_6mm_H5mm")
     )
-    (path "/4cdcdbcd-0741-4981-b73d-143743805270"
-      (reference "SW7") (unit 1) (value "JOYSTICK_BUTTON") (footprint "rf_controller_hw:Joystick_Button")
-    )
     (path "/881ac59d-5f23-4328-9a26-61425ad74be0"
+      (reference "SW7") (unit 1) (value "SW_Push") (footprint "Button_Switch_THT:SW_PUSH_6mm_H5mm")
+    )
+    (path "/7eca3aab-c402-41ce-a461-b675056355b5"
       (reference "SW8") (unit 1) (value "SW_Push") (footprint "Button_Switch_THT:SW_PUSH_6mm_H5mm")
     )
-    (path "/7eca3aab-c402-41ce-a461-b675056355b5"
-      (reference "SW9") (unit 1) (value "SW_Push") (footprint "Button_Switch_THT:SW_PUSH_6mm_H5mm")
-    )
     (path "/477fbc44-c3ee-44cb-a28e-09e0207b9d55"
-      (reference "SW10") (unit 1) (value "SW_SPDT") (footprint "Connector_PinHeader_2.54mm:PinHeader_1x03_P2.54mm_Vertical")
-    )
-  )
+      (reference "SW9") (unit 1) (value "SW_SPDT") (footprint "Connector_PinHeader_2.54mm:PinHeader_1x03_P2.54mm_Vertical")
+    )
+    (path "/691fef37-3035-4bf1-a7e9-ebb9530ca238"
+      (reference "SW10") (unit 1) (value "SW_DIP_x05") (footprint "Button_Switch_THT:SW_DIP_SPSTx05_Slide_9.78x14.88mm_W7.62mm_P2.54mm")
+    )
+  )
